File: 2 Hardware/Schematics/Relay_Module_Basic_Schematic.kicad_sch (KiCad schematic)
At the start: 6 parts

Commit message: Added gitignre, changes (minor) to schematic, changes to horizontal model (WithWheels) and general repo cleanup
Parts:
- D?: value DIODE -> ${SIM.PARAMS}; Spice_Netlist_Enabled Y -> (none); Spice_Primitive D -> (none)
